File: kb45p/kb45p.kicad_pcb (KiCad board)
At the start: 2 copper layers, 245.3 x 75.6 mm, 109 parts, among them CON1 DEBUG_CON, IC1 STM32F042, IC2 MCP1703T_3LEAD, J1 USB_mini_micro_B

Commit message: kb45p: Add CON1 labels and BOM.
Other:
- board text added: "3V3"
- board text added: "CLK"
- board text added: "DIO"
- board text added: "GND"
- board text added: "RST"
Changed lines of the file:
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@@
     (area 37.310624 32.984695 282.729376 108.739376)
     (thickness 1.6)
-    (drawings 12)
+    (drawings 22)
     (tracks 657)
     (zones 0)
@@
       (net 52 "Net-(D1-Pad2)"))
   )
+  (gr_text RST (at 141.37 104.28 90) (layer B.SilkS)
+    (effects (font (size 1.2 1.2) (thickness 0.25)) (justify mirror))
+  )
+  (gr_text DIO (at 143.22 104.28 90) (layer B.SilkS)
+    (effects (font (size 1.2 1.2) (thickness 0.25)) (justify mirror))
+  )
+  (gr_text 3V3 (at 150.82 104.28 90) (layer B.SilkS)
+    (effects (font (size 1.2 1.2) (thickness 0.25)) (justify mirror))
+  )
+  (gr_text CLK (at 148.27 104.23 90) (layer B.SilkS)
+    (effects (font (size 1.2 1.2) (thickness 0.25)) (justify mirror))
+  )
+  (gr_text GND (at 145.77 104.13 90) (layer B.SilkS)
+    (effects (font (size 1.2 1.2) (thickness 0.25)) (justify mirror))
+  )
+  (gr_line (start 144.52 106.98) (end 144.52 108.08) (angle 90) (layer B.SilkS) (width 0.2))
+  (gr_line (start 146.97 106.98) (end 146.97 108.03) (angle 90) (layer B.SilkS) (width 0.2))
+  (gr_line (start 146.27 106.28) (end 146.97 106.98) (angle 90) (layer B.SilkS) (width 0.2))
+  (gr_line (start 145.22 106.28) (end 146.27 106.28) (angle 90) (layer B.SilkS) (width 0.2))
+  (gr_line (start 144.52 106.98) (end 145.22 106.28) (angle 90) (layer B.SilkS) (width 0.2))
   (gr_text "    jan 2016\n(c) flabbergast" (at 264.199871 93.186292) (layer B.SilkS)
     (effects (font (size 1.5 1.5) (thickness 0.3)) (justify mirror))
