File: stm32_qfp48_breakout/stm32_qfp48_breakout.kicad_pcb (KiCad board)
At the start: 2 copper layers, 35.6 x 17.8 mm, 26 parts, among them IC1 STM32L052C8T7, IC2 NCV8170, J1 USB_mini_micro_B, U1 M14, U2 M14, U3 M05, Y1 CRYSTAL

Commit message: STM32-QFP48-breakout rev1.
Routing:
- net GND: track 104.5 -> 113.3 mm, vias 11 -> 13
Other:
- rule pad_to_mask_clearance: 0.2 -> 0.05
- board text added: "a15^"
Changed lines of the file:
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@@
     (links 87)
     (no_connects 1)
-    (area 152.324999 92.634999 188.035001 110.565001)
+    (area 150.338428 90.941398 189.578742 112.108742)
     (thickness 1.6)
-    (drawings 104)
-    (tracks 457)
+    (drawings 105)
+    (tracks 467)
     (zones 0)
     (modules 26)
@@
     (pad_size 1.524 1.524)
     (pad_drill 0.762)
-    (pad_to_mask_clearance 0.2)
+    (pad_to_mask_clearance 0.05)
     (aux_axis_origin 0 0)
     (grid_origin 180.594 107.823)
@@
     )
   )
+  (gr_text a15^ (at 162.179 104.521) (layer F.SilkS)
+    (effects (font (size 0.7 0.7) (thickness 0.127)))
+  )
   (gr_text ss (at 180.848 107.823 315) (layer B.SilkS)
     (effects (font (size 0.7 0.7) (thickness 0.127)) (justify mirror))
@@
   (gr_line (start 152.4 109.855) (end 153.035 110.49) (angle 90) (layer Edge.Cuts) (width 0.15))
   (gr_line (start 152.4 93.345) (end 152.4 109.855) (angle 90) (layer Edge.Cuts) (width 0.15))
+  (segment (start 165.5318 97.9678) (end 166.920201 97.9678) (width 0.25) (layer B.Cu) (net 1))
+  (segment (start 165.50132 97.93732) (end 165.5318 97.9678) (width 0.25) (layer F.Cu) (net 1))
+  (via (at 165.5318 97.9678) (size 0.6858) (drill 0.34) (layers F.Cu B.Cu) (net 1))
+  (segment (start 166.16172 97.30232) (end 165.50132 97.93732) (width 0.25) (layer F.Cu) (net 1))
+  (segment (start 172.862885 97.291515) (end 173.9138 96.393) (width 0.25) (layer B.Cu) (net 1))
+  (via (at 173.9138 96.393) (size 0.6858) (drill 0.34) (layers F.Cu B.Cu) (net 1))
+  (segment (start 173.9138 96.393) (end 174.498 96.8756) (width 0.25) (layer F.Cu) (net 1))
   (segment (start 167.596486 97.291515) (end 172.862885 97.291515) (width 0.25) (layer B.Cu) (net 1))
-  (segment (start 173.9138 96.393) (end 174.498 96.8756) (width 0.25) (layer F.Cu) (net 1))
-  (via (at 173.9138 96.393) (size 0.6858) (drill 0.34) (layers F.Cu B.Cu) (net 1))
-  (segment (start 172.862885 97.291515) (end 173.9138 96.393) (width 0.25) (layer B.Cu) (net 1))
+  (segment (start 166.920201 97.9678) (end 167.596486 97.291515) (width 0.25) (layer B.Cu) (net 1))
   (segment (start 174.498 96.8756) (end 174.498 97.028) (width 0.25) (layer F.Cu) (net 1))
   (segment (start 171.65828 104.42448) (end 171.65828 105.89768) (width 0.25) (layer F.Cu) (net 1))
@@
   (segment (start 177.546 99.5426) (end 175.0314 97.028) (width 0.25) (layer F.Cu) (net 1))
   (segment (start 175.0314 97.028) (end 174.498 97.028) (width 0.25) (layer F.Cu) (net 1))
-  (segment (start 166.16172 97.30232) (end 165.50132 97.93732) (width 0.25) (layer F.Cu) (net 1))
-  (segment (start 165.608 98.044) (end 167.596486 97.291515) (width 0.25) (layer B.Cu) (net 1))
-  (segment (start 167.596486 97.291515) (end 167.692567 97.181949) (width 0.25) (layer B.Cu) (net 1))
-  (segment (start 165.5318 97.9678) (end 165.608 98.044) (width 0.25) (layer B.Cu) (net 1))
-  (via (at 165.5318 97.9678) (size 0.6858) (drill 0.34) (layers F.Cu B.Cu) (net 1))
-  (segment (start 165.50132 97.93732) (end 165.5318 97.9678) (width 0.25) (layer F.Cu) (net 1))
   (segment (start 183.256 104.306) (end 186.651 104.306) (width 0.25) (layer F.Cu) (net 1))
   (segment (start 186.651 104.306) (end 186.817 104.14) (width 0.25) (layer F.Cu) (net 1))
@@
   (segment (start 164.846 106.172) (end 164.846 104.58196) (width 0.25) (layer F.Cu) (net 1))
   (segment (start 164.846 104.58196) (end 164.61232 104.34828) (width 0.25) (layer F.Cu) (net 1))
+  (segment (start 170.688 99.06) (end 171.196 99.06) (width 0.1524) (layer F.Cu) (net 2))
+  (via (at 170.688 99.06) (size 0.6858) (drill 0.34) (layers F.Cu B.Cu) (net 2))
+  (segment (start 170.8658 104.648) (end 170.8658 104.0638) (width 0.1524) (layer B.Cu) (net 2))
+  (via (at 169.926 99.06) (size 0.6858) (drill 0.34) (layers F.Cu B.Cu) (net 2))
+  (segment (start 169.037 99.06) (end 169.926 99.06) (width 0.1524) (layer B.Cu) (net 2))
+  (segment (start 168.656 99.441) (end 169.037 99.06) (width 0.1524) (layer B.Cu) (net 2))
+  (segment (start 168.656 100.965) (end 168.656 99.441) (width 0.1524) (layer B.Cu) (net 2))
+  (segment (start 169.164 101.473) (end 168.656 100.965) (width 0.1524) (layer B.Cu) (net 2))
+  (segment (start 169.164 102.362) (end 169.164 101.473) (width 0.1524) (layer B.Cu) (net 2))
+  (segment (start 170.8658 104.0638) (end 169.164 102.362) (width 0.1524) (layer B.Cu) (net 2))
+  (segment (start 170.688 99.06) (end 169.926 99.06) (width 0.1524) (layer F.Cu) (net 2))
+  (segment (start 171.196 99.06) (end 171.2722 98.9838) (width 0.1524) (layer F.Cu) (net 2))
+  (segment (start 164.61232 103.8479) (end 163.3855 103.8479) (width 0.25) (layer F.Cu) (net 2))
+  (via (at 163.195 103.6574) (size 0.6858) (drill 0.34) (layers F.Cu B.Cu) (net 2))
+  (segment (start 162.7378 104.1146) (end 163.195 103.6574) (width 0.25) (layer B.Cu) (net 2))
+  (segment (start 162.7378 104.1146) (end 162.7378 105.283) (width 0.25) (layer B.Cu) (net 2))
+  (segment (start 163.3855 103.8479) (end 163.195 103.6574) (width 0.25) (layer F.Cu) (net 2))
   (segment (start 159.385 98.795) (end 159.385 99.5172) (width 0.25) (layer F.Cu) (net 2))
   (segment (start 159.385 99.5172) (end 159.5374 99.6696) (width 0.25) (layer F.Cu) (net 2))
@@
   (segment (start 177.5578 98.894) (end 175.3108 96.647) (width 0.25) (layer F.Cu) (net 2))
   (segment (start 173.20768 100.8507) (end 171.8183 100.8507) (width 0.25) (layer F.Cu) (net 2))
+  (segment (start 171.8183 100.8507) (end 171.2722 100.3046) (width 0.25) (layer F.Cu) (net 2))
+  (segment (start 171.2722 100.3046) (end 171.2722 98.9838) (width 0.25) (layer F.Cu) (net 2))
   (segment (start 171.2722 98.9838) (end 172.974 97.282) (width 0.25) (layer F.Cu) (net 2))
-  (segment (start 171.2722 100.3046) (end 171.2722 98.9838) (width 0.25) (layer F.Cu) (net 2))
-  (segment (start 171.8183 100.8507) (end 171.2722 100.3046) (width 0.25) (layer F.Cu) (net 2))
   (segment (start 172.974 97.282) (end 172.974 97.028) (width 0.25) (layer F.Cu) (net 2))
   (segment (start 182.372 100.838) (end 183.642 100.838) (width 0.25) (layer B.Cu) (net 2))
@@
   (via (at 173.99 106.7816) (size 0.6858) (drill 0.34) (layers F.Cu B.Cu) (net 2))
   (segment (start 172.847 105.283) (end 173.99 106.7816) (width 0.25) (layer B.Cu) (net 2))
-  (segment (start 162.7378 105.283) (end 162.7378 104.1146) (width 0.25) (layer B.Cu) (net 2))
-  (segment (start 163.483478 103.945878) (end 164.61232 103.945878) (width 0.25) (layer F.Cu) (net 2))
-  (segment (start 163.195 103.6574) (end 163.483478 103.945878) (width 0.25) (layer F.Cu) (net 2))
-  (via (at 163.195 103.6574) (size 0.6858) (drill 0.34) (layers F.Cu B.Cu) (net 2))
-  (segment (start 162.7378 104.1146) (end 163.195 103.6574) (width 0.25) (layer B.Cu) (net 2))
-  (segment (start 164.61232 103.945878) (end 164.61232 103.8479) (width 0.25) (layer F.Cu) (net 2))
   (segment (start 160.2994 102.8446) (end 162.7378 105.283) (width 0.25) (layer B.Cu) (net 2))
   (segment (start 162.7378 105.283) (end 163.322 105.8672) (width 0.25) (layer F.Cu) (net 2))

Commit message: Update.
Other:
- board text added: "15"
- board text removed: "13"
Changed lines of the file:
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@@
     (effects (font (size 0.89916 0.89916) (thickness 0.14986)))
   )
-  (gr_text 13 (at 184.023 107.569) (layer F.SilkS)
+  (gr_text 15 (at 184.023 107.569) (layer F.SilkS)
     (effects (font (size 0.7 0.7) (thickness 0.127)))
   )

Commit message: Update bat board.
Parts:
- added JP3: BT0, flabbergast:SOLDER_JUMPER_ON, B.Cu at (178.9, 106.1)
- added R3: 1.5kR, flabbergast:0603, B.Cu at (158.3, 105.5)
- C7: footprint flabbergast:0603 -> flabbergast:0603_NOPASTE
- JP1, JP2: footprint flabbergast:SOLDER_JUMPER_OFF -> flabbergast:SOLDER_JUMPER_OFF_PASTE
- moved PAD1 0.05 mm to (156.2, 96.6)
Connections:
- IC1 pad 44: A1(BOOT) -> BOOT0
- R1 pad 1: A1(BOOT) -> BOOT0
- U1 pad 1: VDD -> VIN
- U1 pad 2: VIN -> GND
- U1 pad 3: A9 -> VDD
- U1 pad 4: A10 -> A9
- U1 pad 5: GND -> A10
Routing:
- net BOOT0: track 0.00 -> 14.7 mm, vias 0 -> 4
- net A1(BOOT): track 30.5 -> 21.3 mm, vias 6 -> 2
- net B7: track 4.68 -> 13.6 mm
- net USB_D+: track 8.58 -> 12.8 mm, vias 0 -> 1
- net VDD: track 71.8 -> 68.4 mm
- net VIN: track 10.9 -> 12.4 mm
- net GND: track 113.3 -> 114.6 mm
- net A9: track 10.8 -> 9.54 mm
Other:
- board text added: "STM32-QFP48-breakout a.k.a. the bat board (rev2) (c) 2016 flabbergast"
- board text removed: "STM32-QFP48-breakout a.k.a. the bat board (rev1) (c) 2016 flabbergast"

Commit message: Cleanup and update bat board.
Connections:
- IC1 pad 20: Net-(IC1-Pad20) -> GND
Routing:
- net GND: track 114.6 -> 117.6 mm
Other:
- board text added: "STM32-QFP48-breakout a.k.a. the bat board (rev3) (c) 2017 flabbergast"
- board text removed: "STM32-QFP48-breakout a.k.a. the bat board (rev2) (c) 2016 flabbergast"
