File: stm32_qfp48_breakout/stm32_qfp48_breakout.sch (KiCad schematic (older format))
At the start: 25 parts, among them IC1 STM32L052C8T7, IC2 NCV8170, J1 USB_mini_micro_B, U1 M14, U2 M14, U3 M05, Y1 CRYSTAL

Commit message: STM32-QFP48-breakout rev1.
Parts:
- JP2: footprint flabbergast:SOLDER_JUMPER_ON -> flabbergast:SOLDER_JUMPER_OFF
Changed lines of the file:
@@
 EESchema Schematic File Version 2
 LIBS:flabbergast
-LIBS:SparkFun
 LIBS:stm32_qfp48_breakout-cache
 EELAYER 25 0
@@
 F 0 "JP2" V 2200 2550 50  0000 L BNN
 F 1 "reg" V 2440 2550 50  0000 L BNN
-F 2 "flabbergast:SOLDER_JUMPER_ON" H 2250 2550 60  0001 C CNN
+F 2 "flabbergast:SOLDER_JUMPER_OFF" H 2250 2550 60  0001 C CNN
 F 3 "" H 2250 2550 60  0000 C CNN
 	1    2250 2550

Commit message: Update.
Parts:
- J1: symbol USB_mini_micro_B -> USB_mini_micro_B-RESCUE-stm32_qfp48_breakout
- PAD1: symbol M01 -> M01-RESCUE-stm32_qfp48_breakout
Changed lines of the file:
@@
 EESchema Schematic File Version 2
+LIBS:stm32_qfp48_breakout-rescue
 LIBS:flabbergast
 LIBS:stm32_qfp48_breakout-cache
@@
 $EndComp
 $Comp
-L USB_mini_micro_B J1
+L USB_mini_micro_B-RESCUE-stm32_qfp48_breakout J1
 U 1 1 572321C9
 P 1350 1600
@@
 $EndComp
 $Comp
-L M01 PAD1
+L M01-RESCUE-stm32_qfp48_breakout PAD1
 U 1 1 572328CF
 P 1600 1350

Commit message: Update bat board.
Parts:
- added JP3: BT0, flabbergast:SOLDER_JUMPER_ON, symbol JUMPER-2
- added R3: 1.5kR, flabbergast:0603, symbol RES
- C7: footprint flabbergast:0603 -> flabbergast:0603_NOPASTE
- JP1, JP2: footprint flabbergast:SOLDER_JUMPER_OFF -> flabbergast:SOLDER_JUMPER_OFF_PASTE
Connections:
- net A1(BOOT): now also JP3.2; no longer IC1.44 (BOOT0), R1.1
- net A10: now also U1.5; no longer U1.4
- net A9: now also U1.4; no longer U1.3
- net B7: now also R3.1
- net GND: now also U1.2; no longer U1.5
- net USB_D+: now also R3.2
- net VDD: now also U1.3; no longer U1.1
- net VIN: now also U1.1; no longer U1.2
- new net BOOT0: IC1.44 (BOOT0), JP3.1, R1.1
Other:
- moved on the sheet: R1
Changed lines of the file:
@@
 Title "STM32-QFP48-BREAKOUT"
 Date "29/04/16"
-Rev "rev1"
+Rev "rev2"
 Comp ""
 Comment1 ""
@@
 F 0 "JP1" V 1750 1350 50  0000 L BNN
 F 1 "USB_PWR" V 1990 1350 50  0000 L BNN
-F 2 "flabbergast:SOLDER_JUMPER_OFF" H 1800 1350 60  0001 C CNN
+F 2 "flabbergast:SOLDER_JUMPER_OFF_PASTE" H 1800 1350 60  0001 C CNN
 F 3 "" H 1800 1350 60  0000 C CNN
 	1    1800 1350
@@
 Text GLabel 1700 1550 2    60   Input ~ 0
 USB_D-
-Text GLabel 1700 1650 2    60   Input ~ 0
+Text GLabel 2500 1650 2    60   Input ~ 0
 USB_D+
 NoConn ~ 1500 1750
@@
 F 0 "JP2" V 2200 2550 50  0000 L BNN
 F 1 "reg" V 2440 2550 50  0000 L BNN
-F 2 "flabbergast:SOLDER_JUMPER_OFF" H 2250 2550 60  0001 C CNN
+F 2 "flabbergast:SOLDER_JUMPER_OFF_PASTE" H 2250 2550 60  0001 C CNN
 F 3 "" H 2250 2550 60  0000 C CNN
 	1    2250 2550
@@
 F 0 "C7" H 1860 4215 50  0000 L BNN
 F 1 "1uF" H 1860 4015 50  0000 L BNN
-F 2 "flabbergast:0603" H 1800 4100 60  0001 C CNN
+F 2 "flabbergast:0603_NOPASTE" H 1800 4100 60  0001 C CNN
 F 3 "" H 1800 4100 60  0000 C CNN
 	1    1800 4100
@@
 $EndComp
 Text GLabel 3750 2800 0    60   Input ~ 0
-BOOT_BTN
+BOOT0
 Text GLabel 3750 1450 0    60   Input ~ 0
 RESET_BTN
@@
 Text GLabel 3750 2300 0    60   Input ~ 0
 SWDIO
-Text GLabel 7200 1250 0    60   Input ~ 0
-BOOT_BTN
+Text GLabel 6900 1250 0    60   Input ~ 0
+BOOT0
 $Comp
 L RES R1
 U 1 1 5723450B
-P 7400 1500
-F 0 "R1" V 7480 1500 50  0000 C CNN
-F 1 "10kR" V 7400 1500 50  0000 C CNN
-F 2 "flabbergast:0603" H 7400 1500 60  0001 C CNN
-F 3 "" H 7400 1500 60  0000 C CNN
-	1    7400 1500
+P 7150 1500
+F 0 "R1" V 7230 1500 50  0000 C CNN
+F 1 "10kR" V 7150 1500 50  0000 C CNN
+F 2 "flabbergast:0603" H 7150 1500 60  0001 C CNN
+F 3 "" H 7150 1500 60  0000 C CNN
+	1    7150 1500
 	1    0    0    -1
 $EndComp
@@
 L GND #PWR017
 U 1 1 572345AC
-P 7400 1850
-F 0 "#PWR017" H 7400 1600 50  0001 C CNN
-F 1 "GND" H 7400 1700 50  0000 C CNN
-F 2 "" H 7400 1850 60  0000 C CNN
-F 3 "" H 7400 1850 60  0000 C CNN
-	1    7400 1850
+P 7150 1850
+F 0 "#PWR017" H 7150 1600 50  0001 C CNN
+F 1 "GND" H 7150 1700 50  0000 C CNN
+F 2 "" H 7150 1850 60  0000 C CNN
+F 3 "" H 7150 1850 60  0000 C CNN
+	1    7150 1850
 	1    0    0    -1
 $EndComp
@@
 L VDD #PWR024
 U 1 1 572368FC
+P 10150 1250
+F 0 "#PWR024" H 10150 1100 50  0001 C CNN
+F 1 "VDD" H 10150 1390 50  0000 C CNN
+F 2 "" H 10150 1250 50  0000 C CNN
+F 3 "" H 10150 1250 50  0000 C CNN
+	1    10150 1250
+	1    0    0    -1
+$EndComp
+$Comp
+L VIN #PWR025
+U 1 1 57236948
 P 10300 1250
-F 0 "#PWR024" H 10300 1100 50  0001 C CNN
-F 1 "VDD" H 10300 1390 50  0000 C CNN
+F 0 "#PWR025" H 10300 1100 50  0001 C CNN
+F 1 "VIN" H 10300 1390 50  0000 C CNN
 F 2 "" H 10300 1250 50  0000 C CNN
 F 3 "" H 10300 1250 50  0000 C CNN
@@
 $EndComp
 $Comp
-L VIN #PWR025
-U 1 1 57236948
-P 10150 1350
-F 0 "#PWR025" H 10150 1200 50  0001 C CNN
-F 1 "VIN" H 10150 1490 50  0000 C CNN
-F 2 "" H 10150 1350 50  0000 C CNN
-F 3 "" H 10150 1350 50  0000 C CNN
-	1    10150 1350
-	1    0    0    -1
-$EndComp
-$Comp
 L GND #PWR026
 U 1 1 57236999
-P 9950 1650
-F 0 "#PWR026" H 9950 1400 50  0001 C CNN
-F 1 "GND" H 9950 1500 50  0000 C CNN
-F 2 "" H 9950 1650 60  0000 C CNN
-F 3 "" H 9950 1650 60  0000 C CNN
-	1    9950 1650
-	1    0    0    -1
-$EndComp
-Text GLabel 10300 1450 0    60   Input ~ 0
+P 10050 1350
+F 0 "#PWR026" H 10050 1100 50  0001 C CNN
+F 1 "GND" H 10050 1200 50  0000 C CNN
+F 2 "" H 10050 1350 60  0000 C CNN
+F 3 "" H 10050 1350 60  0000 C CNN
+	1    10050 1350
+	1    0    0    -1
+$EndComp
+Text GLabel 10300 1550 0    60   Input ~ 0
 A9
-Text GLabel 10300 1550 0    60   Input ~ 0
+Text GLabel 10300 1650 0    60   Input ~ 0
 A10
 Text GLabel 10300 1750 0    60   Input ~ 0
@@
 Text GLabel 3750 5300 2    60   Input ~ 0
 OSC_OUT
-Text GLabel 7200 1450 0    60   Input ~ 0
+Text GLabel 6900 1450 0    60   Input ~ 0
 A1(BOOT)
 Text GLabel 9450 2250 2    60   Input ~ 0
@@
 	1    0    0    -1
 $EndComp
-Wire Wire Line
-	7200 1450 7200 1250
 Connection ~ 3600 5300
 Connection ~ 3600 5100
@@
 	10300 1250 10400 1250
 Wire Wire Line
-	10400 1350 10150 1350
-Wire Wire Line
-	10400 1450 10300 1450
+	10050 1350 10400 1350
+Wire Wire Line
+	10150 1450 10400 1450
 Wire Wire Line
 	10300 1550 10400 1550
-Wire Wire Line
-	10400 1650 9950 1650
 Wire Wire Line
 	10300 1750 10400 1750
@@
 Wire Wire Line
 	7600 1250 7600 1150
-Wire Wire Line
-	7400 1750 7400 1850
-Connection ~ 7400 1250
-Wire Wire Line
-	7200 1250 7600 1250
 Wire Wire Line
 	3900 2200 3750 2200
@@
 	1500 1850 1700 1850
 Wire Wire Line
-	1700 1650 1500 1650
+	1500 1650 2500 1650
 Wire Wire Line
 	1500 1550 1700 1550
@@
 Wire Wire Line
 	1500 1450 1800 1450
-Connection ~ 7200 1250
 Text GLabel 5550 2000 2    60   Input ~ 0
 LED
@@
 Wire Wire Line
 	5400 2000 5550 2000
+$Comp
+L JUMPER-2 JP3
+U 1 1 5740521A
+P 7250 1150
+F 0 "JP3" V 7200 1150 50  0000 L BNN
+F 1 "BT0" V 7440 1150 50  0000 L BNN
+F 2 "flabbergast:SOLDER_JUMPER_ON" H 7250 1150 60  0001 C CNN
+F 3 "" H 7250 1150 60  0000 C CNN
+	1    7250 1150
+	1    0    0    -1
+$EndComp
+Wire Wire Line
+	6900 1250 7250 1250
+Wire Wire Line
+	7150 1850 7150 1750
+Connection ~ 7150 1250
+Wire Wire Line
+	7350 1250 7600 1250
+Wire Wire Line
+	6900 1450 7500 1450
+Wire Wire Line
+	7500 1450 7500 1250
+Connection ~ 7500 1250
+Wire Wire Line
+	10300 1650 10400 1650
+Wire Wire Line
+	10150 1450 10150 1250
+$Comp
+L RES R3
+U 1 1 5749E614
+P 2400 1300
+F 0 "R3" V 2480 1300 50  0000 C CNN
+F 1 "1.5kR" V 2400 1300 50  0000 C CNN
+F 2 "flabbergast:0603" H 2400 1300 60  0001 C CNN
+F 3 "" H 2400 1300 60  0000 C CNN
+	1    2400 1300
+	1    0    0    -1
+$EndComp
+Wire Wire Line
+	2400 1550 2400 1650
+Connection ~ 2400 1650
+Wire Wire Line
+	2500 1050 2400 1050
+Text GLabel 2500 1050 2    60   Input ~ 0
+B7
 $EndSCHEMATC

Commit message: Cleanup and update bat board.
Connections:
- net GND: now also IC1.20 (PB2)
- no-connect marks 7 -> 6
Changed lines of the file:
@@
 encoding utf-8
 Sheet 1 1
-Title "STM32-QFP48-BREAKOUT"
-Date "29/04/16"
-Rev "rev2"
-Comp ""
-Comment1 ""
-Comment2 ""
+Title "the bat board: a stm32 qfp48 breakout board"
+Date "2017-10-26"
+Rev "rev3"
+Comp "flabbergast"
+Comment1 "rev2 > rev1: add R3, add JP3, rearrange power pinout"
+Comment2 "rev3 > rev2: connect PB2=BOOT1 to GND"
 Comment3 ""
 Comment4 ""
@@
 NoConn ~ 5400 3250
 NoConn ~ 5400 3150
-NoConn ~ 5400 3050
 Wire Wire Line
 	5550 1250 5400 1250
@@
 Text GLabel 2500 1050 2    60   Input ~ 0
 B7
+$Comp
+L GND #PWR?
+U 1 1 59F1A550
+P 5650 3050
+F 0 "#PWR?" H 5650 2800 50  0001 C CNN
+F 1 "GND" H 5650 2900 50  0000 C CNN
+F 2 "" H 5650 3050 60  0000 C CNN
+F 3 "" H 5650 3050 60  0000 C CNN
+	1    5650 3050
+	1    0    0    -1
+$EndComp
+Wire Wire Line
+	5650 3050 5400 3050
 $EndSCHEMATC
